File: smash.sch (EAGLE design)
At the start: 23 parts, among them U1 MAX232

Commit message: added board files
Parts:
- removed PWR: (no value), nonolith:HEADER-2X3
- added 28VIN, JP1: (no value), nonolith:HEADER-2X3
- added 3V3-I2C, AUXSER, MOT-THRUST: (no value), nonolith:HEADER-1X3ROUND
- added ATXMEGA32A4U: (no value), nonolith:ATXMEGAXXA4U-AU
- added C10, C11, C12, C13, C14, C9: (no value), nonolith:CAP_CERAMIC0603
- added CN1: (no value), nonolith:USBMICROB
- added EXT_I2C: (no value), nonolith:HEADER-1X4ROUND
- added LED1: (no value), microbuilder:LED0603
- added R1, R2, R3, R4: (no value), nonolith:RESISTOR0603
- added RN2, RN3: (no value), nonolith:RNETWORK
- added U$5: MCP1700, nonolith:MCP1700
- added U$6, U$7: M19, SparkFun:M19
- added Y1: (no value), nonolith:CRYSTAL
Connections:
- removed net 5V0: C2.+, C5.P$1, U$3.VIN, U$4.VO
- removed net N$1: ENC0.3, ENC1.3, ENC2.3
- removed net N$3: ENC0.1
- removed net N$4: ENC1.1
- removed net N$5: ENC2.1
- removed net XMEGA-SCL: RN1D.2, U$1.SCL1
- removed net XMEGA-SDA: RN1C.2, U$1.SDA1
- new net 5V: C13.P$1, C14.P$2, C2.+, C5.P$1, CN1.VBUS, ENC0.3, ENC1.3, ENC2.3, U$3.VIN, U$4.VO, U$5.V+, U$6.1, U$6.19
- new net AUX-RX: AUXSER.1, U1.R2IN
- new net AUX-TX: AUXSER.2, U1.T2OUT
- new net ENCO0: ENC0.1, R2.1
- new net ENCO1: ENC1.1, R3.1
- new net ENCO2: ENC2.1, R4.1
- new net N$20: U1.R2OUT
- new net N$21: U1.T2IN
- new net N$6: LED1.C, R1.1
- new net N$9: U1.T1IN
- new net PA0: ATXMEGA32A4U.PA0/ADC0/AREFA, U$6.3
- new net PA1: ATXMEGA32A4U.PA1/ADC1, U$6.4
- new net PA2: ATXMEGA32A4U.PA2/ADC2, U$6.5
- new net PA3: ATXMEGA32A4U.PA3/ADC3, U$6.6
- new net PA4: ATXMEGA32A4U.PA4/ADC4, U$6.7
- new net PA5: ATXMEGA32A4U.PA5/ADC5, U$6.8
- new net PA6: ATXMEGA32A4U.PA6/ADC6, U$6.9
- new net PA7: ATXMEGA32A4U.PA7/ADC7, U$6.10
- new net PB0: ATXMEGA32A4U.PB0/ADC8/AREFB, U$6.11
- new net PB1: ATXMEGA32A4U.PB1/ADC9, U$6.12
- new net PB2: ATXMEGA32A4U.PB2/ADC10/DAC0, U$6.13
- new net PB3: ATXMEGA32A4U.PB3/ADC11/DAC1, U$6.14
- new net PC0: 3V3-I2C.2, ATXMEGA32A4U.PC0/OC0A/SDA, RN1C.2, U$1.SDA1, U$6.15
- new net PC1: 3V3-I2C.3, ATXMEGA32A4U.PC1/OC0B/XCK0/SCL, RN1D.2, U$1.SCL1, U$6.16
- new net PC2: ATXMEGA32A4U.PC2/OC0C/RXD0, U$7.19
- new net PC3: ATXMEGA32A4U.PC3/OC0D/TXD0, U$7.18
- new net PC4: ATXMEGA32A4U.PC4/OC1A/#SS, U$7.17
- new net PC5: ATXMEGA32A4U.PC5/OC1B/MOSI/XCK1, U$7.16
- new net PC6: ATXMEGA32A4U.PC6/MISO/RXD1, U$7.15
- new net PC7: ATXMEGA32A4U.PC7/SCK/TXD1/CLKO/EVO, U$7.14
- new net PD0: ATXMEGA32A4U.OC0A/PD0, R2.2, RN2A.1, U$7.13
- new net PD1: ATXMEGA32A4U.OC0B/XCK0/PD1, R3.2, RN2B.1, U$7.12
- new net PD2: ATXMEGA32A4U.OC0C/RXD0/PD2, R4.2, RN2C.1, U$7.11
- new net PD3: ATXMEGA32A4U.OC0D/TXD0/PD3, U$7.10
- new net PD4: ATXMEGA32A4U.SS/PD4, U$7.9
- new net PD5: ATXMEGA32A4U.XCK1/MOSI/PD5, U$7.8
- new net PDI-CLK: ATXMEGA32A4U.RESET/PDI-CLK, JP1.5
- new net PDI-DATA: ATXMEGA32A4U.PDI-DATA, JP1.1
- new net PE0: ATXMEGA32A4U.OC0A/SDA/PE0, RN3A.2, U$7.7
- new net PE0-P: MOT0.1, RN3A.1
- new net PE1: ATXMEGA32A4U.XCK0/OC0B/SCL/PE1, RN3B.2, U$7.6
- new net PE1-P: MOT1.1, RN3B.1
- new net PE2: ATXMEGA32A4U.RXD0/OC0C/PE2, LED1.A, RN3C.2, U$7.5
- new net PE2-P: MOT2.1, RN3C.1
- new net PE3: ATXMEGA32A4U.TXD0/OC0D/PE3, RN3D.2, U$7.4
- new net PE3-P: MOT-THRUST.1, RN3D.1
- new net PR0: ATXMEGA32A4U.PR0/XTAL2, C11.P$1, Y1.2
- new net PR1: ATXMEGA32A4U.PR1/XTAL1, C12.P$1, Y1.1
- new net USB+: ATXMEGA32A4U.TXD1/USB+/PD7, CN1.D+
- new net USB-: ATXMEGA32A4U.RXD1/MISO/USB-/PD6, CN1.D-
- net 12V: now also C3.+, MOT0.2, MOT1.2, MOT2.2
- net 28V: now also 28VIN.1, 28VIN.3, 28VIN.5; no longer PWR.1, PWR.3, PWR.5
- net 3V3: now also ATXMEGA32A4U.AVCC, ATXMEGA32A4U.VCC@1, ATXMEGA32A4U.VCC@2, ATXMEGA32A4U.VCC@3, C10.P$1, C9.P$1, JP1.2, U$5.VO, U$6.18, U$7.2
- net 4V3: now also EXT_I2C.2
- net GND: now also 28VIN.2, 28VIN.4, 28VIN.6, 3V3-I2C.1, ATXMEGA32A4U.GND@1, ATXMEGA32A4U.GND@2, ATXMEGA32A4U.GND@3, ATXMEGA32A4U.GND@4, AUXSER.3, C10.P$2, C11.P$2, C12.P$2, C13.P$2, C14.P$1, C3.-, C9.P$2, CN1.GND, ENC0.2, ENC1.2, ENC2.2, EXT_I2C.4, JP1.6, MOT-THRUST.3, MOT0.3, MOT1.3, MOT2.3, R1.2, RN2A.2, RN2B.2, RN2C.2, U$5.GND, U$6.17, U$6.2, U$7.1, U$7.3; no longer PWR.2, PWR.4, PWR.6
- net N$2: now also U1.R1OUT; no longer ENC0.2, ENC1.2, ENC2.2
- net NXT-SCL: now also EXT_I2C.1, RN1A.2; no longer RN1B.2
- net NXT-SDA: now also EXT_I2C.3, RN1B.2; no longer RN1A.2
- net REMUS-RX: now also U1.R1IN
- net REMUS-TX: now also U1.T1OUT
